Commit message: Final DH

File: cheeta_pkg_v4/urdf/cheeta_pkg_v4.urdf (robot description, URDF)
Before this commit: robot cheeta_pkg_v4, 13 links, 12 joints
Joints:
- joint abductor2_joint: axis 0 0 1 -> 0 0 -1
- joint abductor3_joint: axis 0 0 -1 -> 0 0 1
- joint abductor4_joint: axis 0 0 1 -> 0 0 -1
- joint muslo2_joint: axis 0.015133259758379 0 -0.999885485667777 -> 0.015133259758379 0 0.999885485667777
- joint tobillo2_joint: origin xyz=0.0258486456049929 0.0925 0.0076 rpy=0 0 1.27 -> xyz=0.0258486456049929 0.0925 0.0076 rpy=0 0 1.570796327

Commit message: Final DH v2

File: cheeta_pkg_v4/urdf/cheeta_pkg_v4.urdf (robot description, URDF)
Before this commit: robot cheeta_pkg_v4, 13 links, 12 joints
Joints:
- joint tobillo2_joint: axis 0 0 -1 -> 0 0 1

Commit message: Revised DH

File: cheeta_pkg_v4/urdf/cheeta_pkg_v4.urdf (robot description, URDF)
Before this commit: robot cheeta_pkg_v4, 13 links, 12 joints
Joints:
- joint muslo2_joint: axis 0.015133259758379 0 0.999885485667777 -> 0.015133259758379 0  0.999885485667777
